File: PCB/Prototype2/Prototype2.kicad_sch (KiCad schematic)
At the start: 93 parts, among them J2 2x20_Conn, J3 Conn_01x03_Pin, Q1 SSM3K72KCT, Q10 SSM3K72KCT, Q11 SSM3K72KCT, Q12 SSM3K72KCT, Q13 SSM3K72KCT, Q14 SSM3K72KCT, Q15 SSM3K72KCT, Q16 SSM3K72KCT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

Commit message: Added several new test boards
Other:
- note added: "A1"
- note added: "A10"
- note added: "A11"
- note added: "A12"
- note added: "A2"
- note added: "A3"
- note added: "A4"
- note added: "A5"
- note added: "A6"
- note added: "A7"
- note added: "B1"
- note added: "B14"
- note added: "C1"
- note added: "C10"
- note added: "C11"
- note added: "C12"
- note added: "C14"
- note added: "C3"
- note added: "C4"
- note added: "C5"
- note added: "C6"
- note added: "C7"
- note added: "C9"
- note added: "D1"
- note added: "D10"
- note added: "D11"
- note added: "D12"
- note added: "D14"
- note added: "D3"
- note added: "D4"
- note added: "D5"
- note added: "D6"
- note added: "D7"
- note added: "D9"
- note added: "E1"
- note added: "E11"
- note added: "E12"
- note added: "E14"
- note added: "E4"
- note added: "F11"
- note added: "F12"
- note added: "F14"
- note added: "F3"
- note added: "F4"
- note added: "G1"
- note added: "G11"
- note added: "G12"
- note added: "G14"
- note added: "G3"
- note added: "G4"
- note added: "H1"
- note added: "H11"
- note added: "H12"
- note added: "H3"
- note added: "H4"
- note added: "J1"
- note added: "J12"
- note added: "J3"
- note added: "K3"
- note added: "K4"
- note added: "L1"
- note added: "M1"
- note added: "N1"
- note added: "P1"
Changed lines of the file:
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@@
     (fill (type none))
   )
+  (text "G12" (at 267.335 128.905 0)
+    (effects (font (size 1.27 1.27)) (justify left bottom))
+  )
+  (text "D7" (at 267.335 116.205 0)
+    (effects (font (size 1.27 1.27)) (justify left bottom))
+  )
+  (text "D5" (at 267.335 106.045 0)
+    (effects (font (size 1.27 1.27)) (justify left bottom))
+  )
+  (text "C9" (at 313.055 118.745 0)
+    (effects (font (size 1.27 1.27)) (justify left bottom))
+  )
+  (text "F11" (at 267.335 126.365 0)
+    (effects (font (size 1.27 1.27)) (justify left bottom))
+  )
+  (text "D10" (at 267.335 118.745 0)
+    (effects (font (size 1.27 1.27)) (justify left bottom))
+  )
+  (text "P1" (at 282.575 90.805 0)
+    (effects (font (size 1.27 1.27)) (justify left bottom))
+  )
+  (text "C7" (at 267.335 113.665 0)
+    (effects (font (size 1.27 1.27)) (justify left bottom))
+  )
+  (text "D6" (at 282.575 116.205 0)
+    (effects (font (size 1.27 1.27)) (justify left bottom))
+  )
+  (text "E12" (at 297.815 126.365 0)
+    (effects (font (size 1.27 1.27)) (justify left bottom))
+  )
+  (text "E14" (at 313.055 126.365 0)
+    (effects (font (size 1.27 1.27)) (justify left bottom))
+  )
+  (text "A5" (at 267.335 108.585 0)
+    (effects (font (size 1.27 1.27)) (justify left bottom))
+  )
+  (text "L1" (at 297.815 90.805 0)
+    (effects (font (size 1.27 1.27)) (justify left bottom))
+  )
+  (text "C14" (at 313.055 123.825 0)
+    (effects (font (size 1.27 1.27)) (justify left bottom))
+  )
+  (text "F3" (at 282.575 100.965 0)
+    (effects (font (size 1.27 1.27)) (justify left bottom))
+  )
   (text "Keyboard IO" (at 73.66 153.67 0)
     (effects (font (size 1.27 1.27)) (justify left bottom))
   )
+  (text "A2" (at 297.815 106.045 0)
+    (effects (font (size 1.27 1.27)) (justify left bottom))
+  )
+  (text "A1" (at 313.055 106.045 0)
+    (effects (font (size 1.27 1.27)) (justify left bottom))
+  )
+  (text "D3" (at 313.055 103.505 0)
+    (effects (font (size 1.27 1.27)) (justify left bottom))
+  )
+  (text "A10" (at 313.055 116.205 0)
+    (effects (font (size 1.27 1.27)) (justify left bottom))
+  )
+  (text "D4" (at 267.335 103.505 0)
+    (effects (font (size 1.27 1.27)) (justify left bottom))
+  )
+  (text "C5" (at 282.575 108.585 0)
+    (effects (font (size 1.27 1.27)) (justify left bottom))
+  )
+  (text "J3" (at 297.815 93.345 0)
+    (effects (font (size 1.27 1.27)) (justify left bottom))
+  )
+  (text "A7" (at 297.815 113.665 0)
+    (effects (font (size 1.27 1.27)) (justify left bottom))
+  )
+  (text "H1" (at 267.335 95.885 0)
+    (effects (font (size 1.27 1.27)) (justify left bottom))
+  )
+  (text "G4" (at 282.575 98.425 0)
+    (effects (font (size 1.27 1.27)) (justify left bottom))
+  )
+  (text "C12" (at 267.335 121.285 0)
+    (effects (font (size 1.27 1.27)) (justify left bottom))
+  )
+  (text "J12" (at 297.815 131.445 0)
+    (effects (font (size 1.27 1.27)) (justify left bottom))
+  )
+  (text "C3" (at 297.815 103.505 0)
+    (effects (font (size 1.27 1.27)) (justify left bottom))
+  )
+  (text "A12" (at 313.055 121.285 0)
+    (effects (font (size 1.27 1.27)) (justify left bottom))
+  )
+  (text "C11" (at 282.575 121.285 0)
+    (effects (font (size 1.27 1.27)) (justify left bottom))
+  )
+  (text "B1" (at 297.815 100.965 0)
+    (effects (font (size 1.27 1.27)) (justify left bottom))
+  )
+  (text "M1" (at 313.055 90.805 0)
+    (effects (font (size 1.27 1.27)) (justify left bottom))
+  )
+  (text "H4" (at 267.335 98.425 0)
+    (effects (font (size 1.27 1.27)) (justify left bottom))
+  )
+  (text "A4" (at 297.815 108.585 0)
+    (effects (font (size 1.27 1.27)) (justify left bottom))
+  )
+  (text "D1" (at 297.815 98.425 0)
+    (effects (font (size 1.27 1.27)) (justify left bottom))
+  )
   (text "Power Supplies" (at 226.06 19.05 0)
     (effects (font (size 1.27 1.27)) (justify left bottom))
   )
+  (text "A6" (at 313.055 113.665 0)
+    (effects (font (size 1.27 1.27)) (justify left bottom))
+  )
   (text "Potentiometer Inputs" (at 69.85 19.685 0)
     (effects (font (size 1.27 1.27)) (justify left bottom))
   )
+  (text "E11" (at 282.575 126.365 0)
+    (effects (font (size 1.27 1.27)) (justify left bottom))
+  )
   (text "Arcade PCB Interface" (at 138.43 83.82 0)
     (effects (font (size 1.27 1.27)) (justify left bottom))
   )
+  (text "C1" (at 313.055 100.965 0)
+    (effects (font (size 1.27 1.27)) (justify left bottom))
+  )
   (text "Data I/O and Tranceiver Enable" (at 138.43 19.05 0)
     (effects (font (size 1.27 1.27)) (justify left bottom))
   )
+  (text "H12" (at 313.055 131.445 0)
+    (effects (font (size 1.27 1.27)) (justify left bottom))
+  )
+  (text "F4" (at 267.335 100.965 0)
+    (effects (font (size 1.27 1.27)) (justify left bottom))
+  )
   (text "Audio Output" (at 85.725 230.505 0)
     (effects (font (size 1.27 1.27)) (justify left bottom))
   )
+  (text "F14" (at 313.055 128.905 0)
+    (effects (font (size 1.27 1.27)) (justify left bottom))
+  )
+  (text "D9" (at 282.575 118.745 0)
+    (effects (font (size 1.27 1.27)) (justify left bottom))
+  )
+  (text "J1" (at 313.055 93.345 0)
+    (effects (font (size 1.27 1.27)) (justify left bottom))
+  )
+  (text "C4" (at 282.575 106.045 0)
+    (effects (font (size 1.27 1.27)) (justify left bottom))
+  )
+  (text "D14" (at 297.815 123.825 0)
+    (effects (font (size 1.27 1.27)) (justify left bottom))
+  )
+  (text "B14" (at 297.815 121.285 0)
+    (effects (font (size 1.27 1.27)) (justify left bottom))
+  )
   (text "Address Inputs" (at 271.145 154.305 0)
     (effects (font (size 1.27 1.27)) (justify left bottom))
   )
+  (text "C6" (at 282.575 113.665 0)
+    (effects (font (size 1.27 1.27)) (justify left bottom))
+  )
+  (text "E1" (at 313.055 98.425 0)
+    (effects (font (size 1.27 1.27)) (justify left bottom))
+  )
   (text "Misc Input" (at 203.835 153.67 0)
     (effects (font (size 1.27 1.27)) (justify left bottom))
   )
+  (text "K4" (at 282.575 93.345 0)
+    (effects (font (size 1.27 1.27)) (justify left bottom))
+  )
+  (text "E4" (at 282.575 103.505 0)
+    (effects (font (size 1.27 1.27)) (justify left bottom))
+  )
+  (text "C10" (at 297.815 118.745 0)
+    (effects (font (size 1.27 1.27)) (justify left bottom))
+  )
+  (text "G11" (at 282.575 131.445 0)
+    (effects (font (size 1.27 1.27)) (justify left bottom))
+  )
+  (text "A3" (at 313.055 108.585 0)
+    (effects (font (size 1.27 1.27)) (justify left bottom))
+  )
+  (text "N1" (at 267.335 90.805 0)
+    (effects (font (size 1.27 1.27)) (justify left bottom))
+  )
+  (text "K3" (at 267.335 93.345 0)
+    (effects (font (size 1.27 1.27)) (justify left bottom))
+  )
+  (text "F12" (at 282.575 128.905 0)
+    (effects (font (size 1.27 1.27)) (justify left bottom))
+  )
+  (text "H3" (at 282.575 95.885 0)
+    (effects (font (size 1.27 1.27)) (justify left bottom))
+  )
+  (text "D12" (at 267.335 123.825 0)
+    (effects (font (size 1.27 1.27)) (justify left bottom))
+  )
   (text "Open Drain Outputs" (at 210.947 84.455 0)
     (effects (font (size 1.27 1.27)) (justify left bottom))
   )
+  (text "H11" (at 267.335 131.445 0)
+    (effects (font (size 1.27 1.27)) (justify left bottom))
+  )
+  (text "G14" (at 297.815 128.905 0)
+    (effects (font (size 1.27 1.27)) (justify left bottom))
+  )
+  (text "D11" (at 282.575 123.825 0)
+    (effects (font (size 1.27 1.27)) (justify left bottom))
+  )
+  (text "G3" (at 297.815 95.885 0)
+    (effects (font (size 1.27 1.27)) (justify left bottom))
+  )
+  (text "A11" (at 297.815 116.205 0)
+    (effects (font (size 1.27 1.27)) (justify left bottom))
+  )
+  (text "G1" (at 313.055 95.885 0)
+    (effects (font (size 1.27 1.27)) (justify left bottom))
+  )
