File: PCB/Through_Hole_Single_Lattice/Through_Hole_Single.kicad_pcb (KiCad board)
At the start: 2 copper layers, 127.5 x 105.4 mm, 33 parts, among them J1 2x20_Conn, Q1 TN2106, Q10 TN2106, Q2 TN2106, Q3 TN2106, Q4 TN2106, Q5 TN2106, Q6 TN2106, Q7 TN2106, Q8 TN2106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

Commit message: Added several new test boards
Routing:
- net _PHI2: track 79.1 -> 94.5 mm, vias 3 -> 4
- net GND: track 850.7 -> 853.2 mm
- net _P4: track 29.8 -> 30.4 mm
